File: _autosave-reverse-polarity-usmallpro.kicad_pcb (KiCad board)
At the start: 2 copper layers, 31 x 31 mm, 8 parts, among them J1 105-1102-001, J2 105-1102-001, J3 105-1102-001, J4 105-1102-001, Q1 AO3401A, Q2 AO3401A, Q3 AO3401A, Q4 AO3401A

Commit message: updated files
Parts:
- Q1, Q2, Q3, Q4: value AO3401A -> SSM3J355R,LF
- moved Q4 19.0 mm to (68.0, 81.0), turned to 270 degrees
- moved Q3 13.5 mm to (58.5, 90.5), turned to 0 degrees
- moved Q2 13.4 mm to (68.0, 100.0), turned to 90 degrees
